Commit message: add joint state controller

File: angle_ax12_model_pkg/urdf/angle_robot_ax12.urdf.xacro (robot description, xacro)
@@ -69,5 +69,5 @@
 		<child link="ang12ax_link2"/>
 		<origin xyz = "0 0.0151 0.061" rpy="0 0 0" />
-		<axis xyz="0 1 0" />
+		<axis xyz="0 -1 0" />
 		<limit effort="5.0" velocity="5.0"/>
 	</joint>
@@ -101,5 +101,5 @@
 		<child link="ang12ax_link3"/>
 		<origin xyz = "0.0 -0.0082 0.08" rpy="0 0 0" />
-		<axis xyz="0 1 0" />
+		<axis xyz="0 -1 0" />
 		<limit effort="5.0" velocity="5.0"/>
 	</joint>
@@ -133,5 +133,5 @@
 		<child link="ang12ax_link4"/>
 		<origin xyz = "0.0 -0.0078 0.12" rpy="0 0 0" />
-		<axis xyz="0 1 0" />
+		<axis xyz="0 -1 0" />
 		<limit effort="5.0" velocity="5.0"/>
 	</joint>
